Commit message: grasping wrench by gf_6, gf_13

File: envs/bolt_wrench/rsc/end-effector/urdf/end-effector.urdf (robot description, URDF)
Before this commit: robot end-effector, 9 links, 8 joints
Joints:
- joint ee_01_left: origin xyz=-0.027 0 0 rpy=0 0 -0.349065850398886 -> xyz=-0.027 0.073 0.0027 rpy=0 0 -0.349065850398886
- joint ee_01_right: origin xyz=0.027 0 0 rpy=0 0 0.349065850398886 -> xyz=0.027 0.073 0.0027 rpy=0 0 0.349065850398886
- joint ee_02_left: origin xyz=-0.027 0 0 rpy=0 0 0 -> xyz=-0.027 0.073 0.0027 rpy=0 0 0
- joint ee_02_right: origin xyz=0.027 0 0 rpy=0 0 0 -> xyz=0.027 0.073 0.0027 rpy=0 0 0
