Commit message: urdf modified

File: envs/bolt_wrench/rsc/bolt/bolt/urdf/bolt.urdf (robot description, URDF)
Before this commit: robot bolt, 4 links, 3 joints
Links:
- link bolt_rev: mass 0.01286 -> 1000

File: envs/bolt_wrench/rsc/wrench/wrench/urdf/wrench.urdf (robot description, URDF)
Before this commit: robot wrench, 1 links, 0 joints
Links:
- link wrench: mass 0.18231 -> 0.21097

Commit message: bolt z+0.066

File: envs/bolt_wrench/rsc/bolt/bolt/urdf/bolt.urdf (robot description, URDF)
Before this commit: robot bolt, 4 links, 3 joints
Joints:
- joint bolt_base_joint: origin xyz=0 0 0 rpy=0 0 0 -> xyz=0 0 0.066 rpy=0 0 0

Commit message: bolt rev grasped

File: envs/bolt_wrench/rsc/bolt/bolt/urdf/bolt.urdf (robot description, URDF)
Before this commit: robot bolt, 4 links, 3 joints
Links:
- link bolt_rev: geometry collision box size=0.0160 0.0080 0.008; collision box size=0.0160 0.0080 0.008
